Commit message: Layout changes

File: urdf/materials.xacro (robot description, xacro)
@@ -1,12 +1,12 @@
 <?xml version="1.0" ?>
 <robot name="scuttle" xmlns:xacro="http://www.ros.org/wiki/xacro" >
-<material name="silver">
-  <color rgba="0.700 0.700 0.700 1.000"/>
-</material>
-<material name="gray">
-  <color rgba="0.250 0.250 0.250 1.000"/>
-</material>
-<material name="blue">
-  <color rgba="0.000 0.000 0.700 1.000"/>
-</material>
+    <material name="silver">
+        <color rgba="0.700 0.700 0.700 1.000"/>
+    </material>
+    <material name="gray">
+        <color rgba="0.250 0.250 0.250 1.000"/>
+    </material>
+    <material name="blue">
+        <color rgba="0.000 0.000 0.700 1.000"/>
+    </material>
 </robot>
