Commit message: Fixing the swivel wheels

File: urdf/scuttle.xacro (robot description, xacro)
@@ -196,5 +196,5 @@
     -->
     <joint name="l_caster_swivel_joint" type="continuous">
-        <origin rpy="0 0 1.570796" xyz="0.149015 0.119015 -0.025468"/>
+        <origin rpy="0 0 0" xyz="0.250250 0.119250 -0.024660"/>
         <parent link="chassis_link"/>
         <child link="l_caster_swivel"/>
@@ -203,19 +203,21 @@
     <link name="l_caster_swivel">
         <inertial>
-            <origin rpy="0 0 0" xyz="-0.0002554502352885568 0.010633952722858359 -0.012968467515129908"/>
+            <origin rpy="0 0 0" xyz="0 0 0"/>
             <mass value="0.02074189648802402"/>
-            <inertia ixx="7e-06" ixy="0.0" ixz="0.0" iyy="8e-06" iyz="1e-06" izz="9e-06"/>
-        </inertial>
-        <visual>
-            <origin rpy="0 0 0" xyz="0.119279 0.254415 -0.059282"/>
-            <geometry>
-                <mesh filename="package://scuttle_description/meshes/r_caster_swivel_1.stl" scale="0.001 0.001 0.001"/>
-            </geometry>
-            <material name="silver"/>
-        </visual>
-        <collision>
-            <origin rpy="0 0 0" xyz="0.119279 0.254415 -0.059282"/>
-            <geometry>
-                <mesh filename="package://scuttle_description/meshes/r_caster_swivel_collision_1.stl" scale="0.001 0.001 0.001"/>
+            <inertia ixx="7e-06" ixy="0.0" ixz="0.0" iyy="8e-06" iyz="0" izz="9e-06"/>
+        </inertial>
+        <visual>
+            <origin rpy="0 0 0" xyz="0 0 0"/>
+            <geometry>
+                <cylinder length="0.016" radius="0.01951" />
+                <!-- <mesh filename="package://scuttle_description/meshes/l_caster_swivel_1.stl" scale="0.001 0.001 0.001"/> -->
+            </geometry>
+            <material name="silver"/>
+        </visual>
+        <collision>
+            <origin rpy="0 0 0" xyz="0 0 0"/>
+            <geometry>
+                <cylinder length="0.016" radius="0.01951" />
+                <!-- <mesh filename="package://scuttle_description/meshes/l_caster_swivel_collision_1.stl" scale="0.001 0.001 0.001"/> -->
             </geometry>
         </collision>
@@ -225,26 +227,28 @@
     -->
     <joint name="l_caster_wheel_joint" type="continuous">
-        <origin rpy="0 0 0" xyz="-0.017792 0.024 -0.034"/>
+        <origin rpy="0 0 0" xyz="-0.02340 0.0 -0.036340"/>
         <parent link="l_caster_swivel"/>
         <child link="l_caster_wheel"/>
-        <axis xyz="1.0 0.0 -0.0"/>
+        <axis xyz="0.0 1.0 0.0"/>
     </joint>
     <link name="l_caster_wheel">
         <inertial>
-            <origin rpy="0 0 0" xyz="0.0160002016389222 -1.6368916427866864e-07 -7.02880924990934e-08"/>
+            <origin rpy="0 0 0" xyz="0.0 0.0 0.0"/>
             <mass value="0.03841110590847018"/>
             <inertia ixx="1.2e-05" ixy="0.0" ixz="-0.0" iyy="7e-06" iyz="0.0" izz="7e-06"/>
         </inertial>
         <visual>
-            <origin rpy="0 0 0" xyz="-0.101223 0.230415 -0.025282"/>
-            <geometry>
-                <mesh filename="package://scuttle_description/meshes/l_caster_wheel_1.stl" scale="0.001 0.001 0.001"/>
+            <origin rpy="1.570796 0 0" xyz="0 0 0"/>
+            <geometry>
+                <cylinder length="0.0230" radius="0.0244" />
+                <!-- <mesh filename="package://scuttle_description/meshes/l_caster_wheel_1.stl" scale="0.001 0.001 0.001"/> -->
             </geometry>
             <material name="blue"/>
         </visual>
         <collision>
-            <origin rpy="0 0 0" xyz="-0.101223 0.230415 -0.025282"/>
-            <geometry>
-                <mesh filename="package://scuttle_description/meshes/l_caster_wheel_collision_1.stl" scale="0.001 0.001 0.001"/>
+            <origin rpy="1.570796 0 0" xyz="0 0 0"/>
+            <geometry>
+                <cylinder length="0.0230" radius="0.0244" />
+                <!-- <mesh filename="package://scuttle_description/meshes/l_caster_wheel_collision_1.stl" scale="0.001 0.001 0.001"/> -->
             </geometry>
         </collision>
@@ -254,26 +258,28 @@
     -->
     <joint name="r_caster_swivel_joint" type="continuous">
-        <origin rpy="0 0 1.570796" xyz="0.149015 -0.119015 -0.025468"/>
+        <origin rpy="0 0 0" xyz="0.250250 -0.119250 -0.024660"/>
         <parent link="chassis_link"/>
         <child link="r_caster_swivel"/>
-        <axis xyz="0.0 -0.0 1.0"/>
+        <axis xyz="0.0 0.0 1.0"/>
     </joint>
     <link name="r_caster_swivel">
         <inertial>
-            <origin rpy="0 0 0" xyz="-0.00025520971284771765 0.010633952722903461 -0.012968467515129777"/>
-            <mass value="0.02074189648802399"/>
-            <inertia ixx="7e-06" ixy="0.0" ixz="0.0" iyy="8e-06" iyz="1e-06" izz="9e-06"/>
-        </inertial>
-        <visual>
-            <origin rpy="0 0 0" xyz="-0.119015 0.254415 -0.059282"/>
-            <geometry>
-                <mesh filename="package://scuttle_description/meshes/l_caster_swivel_1.stl" scale="0.001 0.001 0.001"/>
-            </geometry>
-            <material name="silver"/>
-        </visual>
-        <collision>
-            <origin rpy="0 0 0" xyz="-0.119015 0.254415 -0.059282"/>
-            <geometry>
-                <mesh filename="package://scuttle_description/meshes/l_caster_swivel_collision_1.stl" scale="0.001 0.001 0.001"/>
+            <origin rpy="0 0 0" xyz="0 0 0"/>
+            <mass value="0.02074189648802402"/>
+            <inertia ixx="7e-06" ixy="0.0" ixz="0.0" iyy="8e-06" iyz="0" izz="9e-06"/>
+        </inertial>
+        <visual>
+            <origin rpy="0 0 0" xyz="0 0 0"/>
+            <geometry>
+                <cylinder length="0.016" radius="0.01951" />
+                <!-- <mesh filename="package://scuttle_description/meshes/r_caster_swivel_1.stl" scale="0.001 0.001 0.001"/> -->
+            </geometry>
+            <material name="silver"/>
+        </visual>
+        <collision>
+            <origin rpy="0 0 0" xyz="0 0 0"/>
+            <geometry>
+                <cylinder length="0.016" radius="0.01951" />
+                <!-- <mesh filename="package://scuttle_description/meshes/r_caster_swivel_collision_1.stl" scale="0.001 0.001 0.001"/> -->
             </geometry>
         </collision>
@@ -283,26 +289,28 @@
     -->
     <joint name="r_caster_wheel_joint" type="continuous">
-        <origin rpy="0 0 0" xyz="0.014208 0.024 -0.034"/>
+        <origin rpy="0 0 0" xyz="-0.02340 0.0 -0.036340"/>
         <parent link="r_caster_swivel"/>
         <child link="r_caster_wheel"/>
-        <axis xyz="-1.0 -0.0 0.0"/>
+        <axis xyz="0.0 1.0 0.0"/>
     </joint>
     <link name="r_caster_wheel">
         <inertial>
-            <origin rpy="0 0 0" xyz="-0.016000038883518655 -1.6368920854881175e-07 -7.028809271419911e-08"/>
-            <mass value="0.03841110590847031"/>
-            <inertia ixx="1.2e-05" ixy="-0.0" ixz="0.0" iyy="7e-06" iyz="0.0" izz="7e-06"/>
-        </inertial>
-        <visual>
-            <origin rpy="0 0 0" xyz="0.105071 0.230415 -0.025282"/>
-            <geometry>
-                <mesh filename="package://scuttle_description/meshes/r_caster_wheel_1.stl" scale="0.001 0.001 0.001"/>
+            <origin rpy="0 0 0" xyz="0.0 0.0 0.0"/>
+            <mass value="0.03841110590847018"/>
+            <inertia ixx="1.2e-05" ixy="0.0" ixz="-0.0" iyy="7e-06" iyz="0.0" izz="7e-06"/>
+        </inertial>
+        <visual>
+            <origin rpy="1.570796 0 0" xyz="0 0 0"/>
+            <geometry>
+                <cylinder length="0.0230" radius="0.0244" />
+                <!-- <mesh filename="package://scuttle_description/meshes/l_caster_wheel_1.stl" scale="0.001 0.001 0.001"/> -->
             </geometry>
             <material name="blue"/>
         </visual>
         <collision>
-            <origin rpy="0 0 0" xyz="0.105071 0.230415 -0.025282"/>
-            <geometry>
-                <mesh filename="package://scuttle_description/meshes/r_caster_wheel_collision_1.stl" scale="0.001 0.001 0.001"/>
+            <origin rpy="1.570796 0 0" xyz="0 0 0"/>
+            <geometry>
+                <cylinder length="0.0230" radius="0.0244" />
+                <!-- <mesh filename="package://scuttle_description/meshes/l_caster_wheel_collision_1.stl" scale="0.001 0.001 0.001"/> -->
             </geometry>
         </collision>
@@ -312,5 +320,5 @@
     -->
     <joint name="lidar" type="fixed">
-        <origin rpy="0 0 3.141592" xyz="-0.077900 0.0 0.024850"/>
+        <origin rpy="0 0 3.141592" xyz="-0.047900 0.0 0.024850"/>
         <parent link="chassis_link"/>
         <child link="lidar_1"/>

Commit message: Comma's in urdf bad

File: urdf/scuttle.xacro (robot description, xacro)
@@ -54,5 +54,5 @@
             <geometry>
                 <!-- <mesh filename="package://scuttle_description/meshes/chassis_link.stl" scale="0.001 0.001 0.001"/> -->
-                <box size="0.365, 0.305, 0.0300" />
+                <box size="0.365 0.305 0.0300" />
             </geometry>
             <material name="silver"/>
@@ -62,5 +62,5 @@
             <geometry>
                 <!-- <mesh filename="package://scuttle_description/meshes/chassis_link_collision.stl" scale="0.001 0.001 0.001"/> -->
-                <box size="0.365, 0.305, 0.0300" />
+                <box size="0.365 0.305 0.0300" />
             </geometry>
         </collision>
@@ -70,5 +70,5 @@
             <geometry>
                 <!-- <mesh filename="package://scuttle_description/meshes/chassis_link.stl" scale="0.001 0.001 0.001"/> -->
-                <box size="0.100, 0.0429, 0.0720" />
+                <box size="0.100 0.0429 0.0720" />
             </geometry>
             <material name="silver"/>
@@ -78,5 +78,5 @@
             <geometry>
                 <!-- <mesh filename="package://scuttle_description/meshes/chassis_link_collision.stl" scale="0.001 0.001 0.001"/> -->
-                <box size="0.100, 0.0429, 0.0720" />
+                <box size="0.100 0.0429 0.0720" />
             </geometry>
         </collision>
@@ -86,5 +86,5 @@
             <geometry>
                 <!-- <mesh filename="package://scuttle_description/meshes/chassis_link.stl" scale="0.001 0.001 0.001"/> -->
-                <box size="0.037, 0.0645, 0.0370" />
+                <box size="0.037 0.0645 0.0370" />
             </geometry>
             <material name="silver"/>
@@ -94,5 +94,5 @@
             <geometry>
                 <!-- <mesh filename="package://scuttle_description/meshes/chassis_link_collision.stl" scale="0.001 0.001 0.001"/> -->
-                <box size="0.037, 0.0645, 0.0370" />
+                <box size="0.037 0.0645 0.0370" />
             </geometry>
         </collision>
@@ -102,5 +102,5 @@
             <geometry>
                 <!-- <mesh filename="package://scuttle_description/meshes/chassis_link.stl" scale="0.001 0.001 0.001"/> -->
-                <box size="0.100, 0.0429, 0.0720" />
+                <box size="0.100 0.0429 0.0720" />
             </geometry>
             <material name="silver"/>
@@ -110,5 +110,5 @@
             <geometry>
                 <!-- <mesh filename="package://scuttle_description/meshes/chassis_link_collision.stl" scale="0.001 0.001 0.001"/> -->
-                <box size="0.100, 0.0429, 0.0720" />
+                <box size="0.100 0.0429 0.0720" />
             </geometry>
         </collision>
@@ -118,5 +118,5 @@
             <geometry>
                 <!-- <mesh filename="package://scuttle_description/meshes/chassis_link.stl" scale="0.001 0.001 0.001"/> -->
-                <box size="0.037, 0.0645, 0.0370" />
+                <box size="0.037 0.0645 0.0370" />
             </geometry>
             <material name="silver"/>
@@ -126,5 +126,5 @@
             <geometry>
                 <!-- <mesh filename="package://scuttle_description/meshes/chassis_link_collision.stl" scale="0.001 0.001 0.001"/> -->
-                <box size="0.037, 0.0645, 0.0370" />
+                <box size="0.037 0.0645 0.0370" />
             </geometry>
         </collision>

Commit message: Fix the initial height

File: urdf/scuttle.xacro (robot description, xacro)
@@ -35,5 +35,5 @@
     -->
     <joint name="chassis_joint" type="fixed">
-        <origin rpy="0 0 0" xyz="0 0 0.095805"/>
+        <origin rpy="0 0 0" xyz="0 0 0.08475"/>
         <parent link="base_link"/>
         <child link="chassis_link"/>

Commit message: tweak the rotation direction for the right wheel

File: urdf/scuttle.xacro (robot description, xacro)
@@ -167,5 +167,5 @@
         <parent link="chassis_link"/>
         <child link="r_wheel"/>
-        <axis xyz="0.0 -1.0 0.0"/>
+        <axis xyz="0.0 1.0 0.0"/>
     </joint>
     <link name="r_wheel">
